Commit message: setting properties to be able to include laser calib date

File: raw_description/urdf/base_long/base.urdf.xacro (robot description, xacro)
@@ -36,8 +36,15 @@
   <property name="battery_size_y" value="0.148" />
   <property name="battery_size_z" value="0.26" />
-  <property name="base_laser_x" value="0.465" />
-  <property name="base_laser_y_back" value="0.23" />
-  <property name="base_laser_y_front" value="0.232" />
+<!--
+  <property name="base_laser_front_x" value="0.465" />
+  <property name="base_laser_rear_x" value="-0.465" />
+  <property name="base_laser_rear_y" value="0.23" />
+  <property name="base_laser_front_y" value="-0.232" />
   <property name="base_laser_z" value="0.178" />
+  <property name="base_laser_yaw_front" value="-M_PI/4" />
+  <property name="base_laser_yaw_rear" value="-5/4*M_PI" />
+  <property name="base_laser_front_yaw" value="-0.785398" />
+  <property name="base_laser_rear_yaw" value="-3.92699" />
+-->
   <!--                                                      -->
   <!--           wheel                                      -->
@@ -195,9 +202,9 @@
     <!-- base laser front -->
     <xacro:sick_s300_laser_v0 name="${name}_laser_front" parent="${name}" ros_topic="scan_front_raw" update_rate="10" min_angle="-2.3562" max_angle="2.3562" >
-      <origin xyz="${base_laser_x} ${-base_laser_y_front} ${base_laser_z}" rpy="${M_PI} 0 ${-M_PI/4}" />
+      <origin xyz="${base_laser_front_x} ${base_laser_front_y} ${base_laser_z}" rpy="${M_PI} 0 ${base_laser_front_yaw}" />
     </xacro:sick_s300_laser_v0>
     <!-- base laser rear -->
     <xacro:sick_s300_laser_v0 name="${name}_laser_rear" parent="${name}" ros_topic="scan_rear_raw" update_rate="10" min_angle="-2.3562" max_angle="2.3562" >
-      <origin xyz="${-base_laser_x} ${base_laser_y_back} ${base_laser_z}" rpy="${M_PI} 0 ${-5*M_PI/4}" />
+      <origin xyz="${base_laser_rear_x} ${base_laser_rear_y} ${base_laser_z}" rpy="${M_PI} 0 ${base_laser_rear_yaw}" />
     </xacro:sick_s300_laser_v0>
     <!-- battery front-->
